Commit message: fix mistakes and prepare for simulation

File: config/moveit/rbs_arm.srdf.xacro (robot description, xacro)
@@ -3,5 +3,8 @@
   <xacro:arg name="name" default="rbs_arm_manip" />
   <xacro:arg name="prefix" default="" />
+  <xacro:arg name="with_gripper" default="false" />
+  <xacro:arg name="gripper_name" default="" />
   <xacro:include filename="$(find rbs_arm)/config/moveit/rbs_arm_macro.srdf.xacro" />
-  <xacro:rbs_arm name="$(arg name)" prefix="$(arg prefix)" />
+  <xacro:rbs_arm name="$(arg name)" prefix="$(arg prefix)" with_gripper="$(arg with_gripper)"
+    gripper_name="$(arg gripper_name)" />
 </robot>

File: config/moveit/rbs_arm_macro.srdf.xacro (robot description, xacro)
@@ -1,24 +1,21 @@
 <?xml version="1.0" encoding="UTF-8"?>
 <robot xmlns:xacro="http://wiki.ros.org/xacro">
-  <xacro:macro name="rbs_arm" params="prefix name">
+  <xacro:macro name="rbs_arm" params="prefix name with_gripper gripper_name">
     <group name="${name}">
-      <chain base_link="${prefix}base_link" tip_link="${prefix}tool0" />
-      <!-- <joint name="${prefix}base_link_joint"/> -->
-      <!-- <joint name="${prefix}fork0_link_joint" /> -->
-      <!-- <joint name="${prefix}main0_link_joint" /> -->
-      <!-- <joint name="${prefix}fork1_link_joint" /> -->
-      <!-- <joint name="${prefix}main1_link_joint" /> -->
-      <!-- <joint name="${prefix}fork2_link_joint" /> -->
-      <!-- <joint name="${prefix}ee_link_joint" /> -->
-      <!-- <joint name="${prefix}tool0_joint" /> -->
+      <xacro:unless value="${with_gripper}">
+        <chain base_link="${prefix}base_link" tip_link="${prefix}tool0" />
+      </xacro:unless>
+      <xacro:if value="${with_gripper}">
+        <chain base_link="${prefix}base_link" tip_link="${prefix}gripper_grasp_point" />
+      </xacro:if>
     </group>
-    <group_state name="home" group="${name}">
-      <joint name="${prefix}ee_link_joint" value="0" />
-      <joint name="${prefix}fork0_link_joint" value="0" />
-      <joint name="${prefix}fork1_link_joint" value="0" />
-      <joint name="${prefix}fork2_link_joint" value="0" />
-      <joint name="${prefix}main0_link_joint" value="0" />
-      <joint name="${prefix}main1_link_joint" value="0" />
-    </group_state>
+    <!-- <group_state name="home" group="${name}"> -->
+    <!--   <joint name="${prefix}ee_link_joint" value="0" /> -->
+    <!--   <joint name="${prefix}fork0_link_joint" value="0" /> -->
+    <!--   <joint name="${prefix}fork1_link_joint" value="0" /> -->
+    <!--   <joint name="${prefix}fork2_link_joint" value="0" /> -->
+    <!--   <joint name="${prefix}main0_link_joint" value="0" /> -->
+    <!--   <joint name="${prefix}main1_link_joint" value="0" /> -->
+    <!-- </group_state> -->
     <disable_collisions link1="${prefix}base_link" link2="${prefix}fork0_link" reason="Adjacent" />
     <disable_collisions link1="${prefix}ee_link" link2="${prefix}fork2_link" reason="Adjacent" />
@@ -33,4 +30,14 @@
     <disable_collisions link1="${prefix}fork2_link" link2="${prefix}main1_link"
       reason="Adjacent" />
+    <disable_collisions link1="${prefix}ee_link" link2="${prefix}${gripper_name}_gripper_base_link"
+      reason="Adjacent" />
+    <disable_collisions link1="${prefix}${gripper_name}_rot_base_link"
+      link2="${prefix}${gripper_name}_l_finger_link" reason="Adjacent" />
+    <disable_collisions link1="${prefix}${gripper_name}_rot_base_link"
+      link2="${prefix}${gripper_name}_r_finger_link" reason="Adjacent" />
+    <disable_collisions link1="${prefix}${gripper_name}_rot_base_link"
+      link2="${prefix}${gripper_name}_gripper_base_link" reason="Adjacent" />
+    <disable_collisions link1="${prefix}${gripper_name}_r_finger_link"
+      link2="${prefix}${gripper_name}_l_finger_link" reason="Adjacent" />
   </xacro:macro>
 </robot>

File: urdf/inc/rbs_fork_link.xacro (robot description, xacro)
@@ -4,5 +4,5 @@
     <xacro:include filename="$(find rbs_arm)/urdf/inc/joint_hardware.xacro" />
     <xacro:include filename="$(find rbs_arm)/urdf/inc/materials.xacro" />
-    <joint name="${prefix}${name}_joint" type="revolute">
+    <joint name="${prefix}${name}_joint" type="continuous">
       <limit lower="-3.14159" upper="3.14159" effort="78" velocity="0.52" />
       <xacro:if value="${parent=='base_link'}">

File: urdf/inc/rbs_main_link.xacro (robot description, xacro)
@@ -4,5 +4,5 @@
     <xacro:include filename="$(find rbs_arm)/urdf/inc/joint_hardware.xacro" />
     <xacro:include filename="$(find rbs_arm)/urdf/inc/materials.xacro"/>
-    <joint name="${prefix}${name}_joint" type="continuous">
+    <joint name="${prefix}${name}_joint" type="revolute">
       <limit lower="-1.5708" upper="3.14159" effort="78" velocity="0.52" />
       <origin rpy="-0.00000 0.00000 0.00000" xyz="0.10000 0.00000 0.09400" />

Commit message: prefix to tf prefix and rework launch files

File: config/moveit/rbs_arm.srdf.xacro (robot description, xacro)
@@ -2,9 +2,9 @@
 <robot xmlns:xacro="http://wiki.ros.org/xacro" name="$(arg name)">
   <xacro:arg name="name" default="rbs_arm_manip" />
-  <xacro:arg name="prefix" default="" />
+  <xacro:arg name="tf_prefix" default="" />
   <xacro:arg name="with_gripper" default="false" />
   <xacro:arg name="gripper_name" default="" />
   <xacro:include filename="$(find rbs_arm)/config/moveit/rbs_arm_macro.srdf.xacro" />
-  <xacro:rbs_arm name="$(arg name)" prefix="$(arg prefix)" with_gripper="$(arg with_gripper)"
+  <xacro:rbs_arm name="$(arg name)" tf_prefix="$(arg tf_prefix)" with_gripper="$(arg with_gripper)"
     gripper_name="$(arg gripper_name)" />
 </robot>

File: config/moveit/rbs_arm_macro.srdf.xacro (robot description, xacro)
@@ -1,43 +1,43 @@
 <?xml version="1.0" encoding="UTF-8"?>
 <robot xmlns:xacro="http://wiki.ros.org/xacro">
-  <xacro:macro name="rbs_arm" params="prefix name with_gripper gripper_name">
+  <xacro:macro name="rbs_arm" params="tf_prefix name with_gripper gripper_name">
     <group name="${name}">
       <xacro:unless value="${with_gripper}">
-        <chain base_link="${prefix}base_link" tip_link="${prefix}tool0" />
+        <chain base_link="${tf_prefix}base_link" tip_link="${tf_prefix}tool0" />
       </xacro:unless>
       <xacro:if value="${with_gripper}">
-        <chain base_link="${prefix}base_link" tip_link="${prefix}gripper_grasp_point" />
+        <chain base_link="${tf_prefix}base_link" tip_link="${tf_prefix}gripper_grasp_point" />
       </xacro:if>
     </group>
     <!-- <group_state name="home" group="${name}"> -->
-    <!--   <joint name="${prefix}ee_link_joint" value="0" /> -->
-    <!--   <joint name="${prefix}fork0_link_joint" value="0" /> -->
-    <!--   <joint name="${prefix}fork1_link_joint" value="0" /> -->
-    <!--   <joint name="${prefix}fork2_link_joint" value="0" /> -->
-    <!--   <joint name="${prefix}main0_link_joint" value="0" /> -->
-    <!--   <joint name="${prefix}main1_link_joint" value="0" /> -->
+    <!--   <joint name="${tf_prefix}ee_link_joint" value="0" /> -->
+    <!--   <joint name="${tf_prefix}fork0_link_joint" value="0" /> -->
+    <!--   <joint name="${tf_prefix}fork1_link_joint" value="0" /> -->
+    <!--   <joint name="${tf_prefix}fork2_link_joint" value="0" /> -->
+    <!--   <joint name="${tf_prefix}main0_link_joint" value="0" /> -->
+    <!--   <joint name="${tf_prefix}main1_link_joint" value="0" /> -->
     <!-- </group_state> -->
-    <disable_collisions link1="${prefix}base_link" link2="${prefix}fork0_link" reason="Adjacent" />
-    <disable_collisions link1="${prefix}ee_link" link2="${prefix}fork2_link" reason="Adjacent" />
-    <disable_collisions link1="${prefix}fork0_link" link2="${prefix}fork1_link" reason="Never" />
-    <disable_collisions link1="${prefix}fork0_link" link2="${prefix}main0_link"
+    <disable_collisions link1="${tf_prefix}base_link" link2="${tf_prefix}fork0_link" reason="Adjacent" />
+    <disable_collisions link1="${tf_prefix}ee_link" link2="${tf_prefix}fork2_link" reason="Adjacent" />
+    <disable_collisions link1="${tf_prefix}fork0_link" link2="${tf_prefix}fork1_link" reason="Never" />
+    <disable_collisions link1="${tf_prefix}fork0_link" link2="${tf_prefix}main0_link"
       reason="Adjacent" />
-    <disable_collisions link1="${prefix}fork1_link" link2="${prefix}fork2_link" reason="Never" />
-    <disable_collisions link1="${prefix}fork1_link" link2="${prefix}main0_link"
+    <disable_collisions link1="${tf_prefix}fork1_link" link2="${tf_prefix}fork2_link" reason="Never" />
+    <disable_collisions link1="${tf_prefix}fork1_link" link2="${tf_prefix}main0_link"
       reason="Adjacent" />
-    <disable_collisions link1="${prefix}fork1_link" link2="${prefix}main1_link"
+    <disable_collisions link1="${tf_prefix}fork1_link" link2="${tf_prefix}main1_link"
       reason="Adjacent" />
-    <disable_collisions link1="${prefix}fork2_link" link2="${prefix}main1_link"
+    <disable_collisions link1="${tf_prefix}fork2_link" link2="${tf_prefix}main1_link"
       reason="Adjacent" />
-    <disable_collisions link1="${prefix}ee_link" link2="${prefix}${gripper_name}_gripper_base_link"
+    <disable_collisions link1="${tf_prefix}ee_link" link2="${tf_prefix}${gripper_name}_gripper_base_link"
       reason="Adjacent" />
-    <disable_collisions link1="${prefix}${gripper_name}_rot_base_link"
-      link2="${prefix}${gripper_name}_l_finger_link" reason="Adjacent" />
-    <disable_collisions link1="${prefix}${gripper_name}_rot_base_link"
-      link2="${prefix}${gripper_name}_r_finger_link" reason="Adjacent" />
-    <disable_collisions link1="${prefix}${gripper_name}_rot_base_link"
-      link2="${prefix}${gripper_name}_gripper_base_link" reason="Adjacent" />
-    <disable_collisions link1="${prefix}${gripper_name}_r_finger_link"
-      link2="${prefix}${gripper_name}_l_finger_link" reason="Adjacent" />
+    <disable_collisions link1="${tf_prefix}${gripper_name}_rot_base_link"
+      link2="${tf_prefix}${gripper_name}_l_finger_link" reason="Adjacent" />
+    <disable_collisions link1="${tf_prefix}${gripper_name}_rot_base_link"
+      link2="${tf_prefix}${gripper_name}_r_finger_link" reason="Adjacent" />
+    <disable_collisions link1="${tf_prefix}${gripper_name}_rot_base_link"
+      link2="${tf_prefix}${gripper_name}_gripper_base_link" reason="Adjacent" />
+    <disable_collisions link1="${tf_prefix}${gripper_name}_r_finger_link"
+      link2="${tf_prefix}${gripper_name}_l_finger_link" reason="Adjacent" />
   </xacro:macro>
 </robot>

File: urdf/inc/joint_interface.xacro (robot description, xacro)
@@ -2,5 +2,5 @@
 <robot xmlns:xacro="http://www.ros.org/wiki/xacro">
         <!-- Individual joint. -->
-        <xacro:macro name="joint_interface" params="name p d">
+  <xacro:macro name="joint_interface" params="name p:=^ d:=^">
                 <joint name="${name}">
                         <command_interface name="position">
@@ -12,6 +12,6 @@
                                 <param name="max">1</param>
                         </command_interface>
-                        <param name="p">${p}</param>
-                        <param name="d">${d}</param>
+                        <!-- <param name="p">${p}</param> -->
+                        <!-- <param name="d">${d}</param> -->
                         <state_interface name="position"/>
                         <state_interface name="velocity"/>

File: urdf/inc/rbs_base_link.xacro (robot description, xacro)
@@ -1,14 +1,14 @@
 <?xml version="1.0" encoding="UTF-8"?>
 <robot xmlns:xacro="http://www.ros.org/wiki/xacro">
-  <xacro:macro name="base_link" params="parent prefix *origin hardware">
+  <xacro:macro name="base_link" params="parent tf_prefix *origin hardware">
     <xacro:include filename="$(find rbs_arm)/urdf/inc/joint_hardware.xacro" />
     <xacro:include filename="$(find rbs_arm)/urdf/inc/materials.xacro"/>
-    <joint name="${prefix}base_link_joint" type="fixed">
+    <joint name="${tf_prefix}base_link_joint" type="fixed">
       <xacro:insert_block name="origin" />
       <parent link="${parent}" />
-      <child link="${prefix}base_link" />
+      <child link="${tf_prefix}base_link" />
     </joint>
-    <link name="${prefix}base_link">
-      <collision name="${prefix}base_link_collision">
+    <link name="${tf_prefix}base_link">
+      <collision name="${tf_prefix}base_link_collision">
         <origin rpy="0.00000 0.00000 0.00000" xyz="0.00000 0.00000 0.00000" />
         <geometry>
@@ -24,5 +24,5 @@
         <mass value="1.88031044620482" />
       </inertial>
-      <visual name="${prefix}base_link_visual">
+      <visual name="${tf_prefix}base_link_visual">
         <origin rpy="0.00000 0.00000 0.00000" xyz="0.00000 0.00000 0.00000" />
         <geometry>
@@ -32,6 +32,6 @@
       </visual>
     </link>
-    <!-- <xacro:joint_hardware joint_name="${prefix}base_link" hardware="${hardware}" p="100"/> -->
-    <xacro:rbs_materials link_name="${prefix}base_link" link_type="base_link" />
+    <!-- <xacro:joint_hardware joint_name="${tf_prefix}base_link" hardware="${hardware}" p="100"/> -->
+    <xacro:rbs_materials link_name="${tf_prefix}base_link" link_type="base_link" />
   </xacro:macro>
 </robot>

File: urdf/inc/rbs_ee_link.xacro (robot description, xacro)
@@ -1,22 +1,22 @@
 <?xml version="1.0" encoding="UTF-8"?>
 <robot xmlns:xacro="http://www.ros.org/wiki/xacro">
-  <xacro:macro name="ee_link" params="prefix parent hardware">
+  <xacro:macro name="ee_link" params="tf_prefix parent hardware">
     <xacro:include filename="$(find rbs_arm)/urdf/inc/joint_hardware.xacro" />
     <xacro:include filename="$(find rbs_arm)/urdf/inc/materials.xacro" />
-    <joint name="${prefix}ee_link_joint" type="revolute">
+    <joint name="${tf_prefix}ee_link_joint" type="revolute">
       <limit lower="-1.5708" upper="3.14159" effort="78" velocity="0.52" />
       <origin rpy="0.00000 0.00000 0.00000" xyz="0.10000 0.00000 0.09473" />
-      <parent link="${prefix}${parent}" />
-      <child link="${prefix}ee_link" />
+      <parent link="${tf_prefix}${parent}" />
+      <child link="${tf_prefix}ee_link" />
       <axis xyz="0 1 0" />
     </joint>
-    <joint name="${prefix}tool0_joint" type="fixed">
+    <joint name="${tf_prefix}tool0_joint" type="fixed">
       <origin rpy="0.00000 0.00000 0.00000" xyz="0.00000 0.00000 0.11000" />
-      <parent link="${prefix}ee_link" />
-      <child link="${prefix}tool0" />
+      <parent link="${tf_prefix}ee_link" />
+      <child link="${tf_prefix}tool0" />
     </joint>
-    <link name="${prefix}tool0" />
-    <link name="${prefix}ee_link">
-      <collision name="${prefix}ee_link_collision">
+    <link name="${tf_prefix}tool0" />
+    <link name="${tf_prefix}ee_link">
+      <collision name="${tf_prefix}ee_link_collision">
         <origin rpy="-0.00000 0.00000 -0.00000" xyz="0.00000 -0.00000 0.00000" />
         <geometry>
@@ -32,5 +32,5 @@
         <mass value="1.88031044620482" />
       </inertial>
-      <visual name="${prefix}ee_link_visual">
+      <visual name="${tf_prefix}ee_link_visual">
         <origin rpy="0.00000 0.00000 0.00000" xyz="0.00000 -0.00000 0.00000" />
         <geometry>
@@ -40,6 +40,6 @@
       </visual>
     </link>
-    <xacro:joint_hardware joint_name="${prefix}ee_link_joint" hardware="${hardware}" p="10" d="0.5" />
-    <xacro:rbs_materials link_name="${prefix}ee_link" link_type="ee_link" />
+    <xacro:joint_hardware joint_name="${tf_prefix}ee_link_joint" hardware="${hardware}" p="10" d="0.5" />
+    <xacro:rbs_materials link_name="${tf_prefix}ee_link" link_type="ee_link" />
   </xacro:macro>
 </robot>

File: urdf/inc/rbs_fork_link.xacro (robot description, xacro)
@@ -1,8 +1,8 @@
 <?xml version="1.0" encoding="UTF-8"?>
 <robot xmlns:xacro="http://www.ros.org/wiki/xacro">
-  <xacro:macro name="fork_link" params="prefix parent name hardware">
+  <xacro:macro name="fork_link" params="tf_prefix parent name hardware">
     <xacro:include filename="$(find rbs_arm)/urdf/inc/joint_hardware.xacro" />
     <xacro:include filename="$(find rbs_arm)/urdf/inc/materials.xacro" />
-    <joint name="${prefix}${name}_joint" type="continuous">
+    <joint name="${tf_prefix}${name}_joint" type="continuous">
       <limit lower="-3.14159" upper="3.14159" effort="78" velocity="0.52" />
       <xacro:if value="${parent=='base_link'}">
@@ -12,10 +12,10 @@
         <origin rpy="0.00000 0.00000 0.00000" xyz="0.00000 0.00000 0.13300" />
       </xacro:unless>
-      <parent link="${prefix}${parent}" />
-      <child link="${prefix}${name}" />
+      <parent link="${tf_prefix}${parent}" />
+      <child link="${tf_prefix}${name}" />
       <axis xyz="0 0 1" />
     </joint>
-    <link name="${prefix}${name}">
-      <collision name="${prefix}${name}_collision">
+    <link name="${tf_prefix}${name}">
+      <collision name="${tf_prefix}${name}_collision">
         <origin rpy="0.00000 0.00000 0.00000" xyz="0.00000 -0.00000 0.00000" />
         <geometry>
@@ -31,5 +31,5 @@
         <mass value="1.12472202892859" />
       </inertial>
-      <visual name="${prefix}${name}_visual">
+      <visual name="${tf_prefix}${name}_visual">
         <origin rpy="0.00000 -0.00000 -0.00000" xyz="0.00000 -0.00000 0.00000" />
         <geometry>
@@ -39,6 +39,6 @@
       </visual>
     </link>
-    <xacro:joint_hardware joint_name="${prefix}${name}_joint" hardware="${hardware}" p="1000000" d="0.5" />
-    <xacro:rbs_materials link_name="${prefix}${name}" link_type="fork" />
+    <xacro:joint_hardware joint_name="${tf_prefix}${name}_joint" hardware="${hardware}" p="1000000" d="0.5" />
+    <xacro:rbs_materials link_name="${tf_prefix}${name}" link_type="fork" />
   </xacro:macro>
 </robot>

File: urdf/inc/rbs_main_link.xacro (robot description, xacro)
@@ -1,16 +1,16 @@
 <?xml version="1.0" encoding="UTF-8"?>
 <robot xmlns:xacro="http://www.ros.org/wiki/xacro">
-  <xacro:macro name="main_link" params="prefix parent name hardware">
+  <xacro:macro name="main_link" params="tf_prefix parent name hardware">
     <xacro:include filename="$(find rbs_arm)/urdf/inc/joint_hardware.xacro" />
-    <xacro:include filename="$(find rbs_arm)/urdf/inc/materials.xacro"/>
-    <joint name="${prefix}${name}_joint" type="revolute">
+    <xacro:include filename="$(find rbs_arm)/urdf/inc/materials.xacro" />
+    <joint name="${tf_prefix}${name}_joint" type="revolute">
       <limit lower="-1.5708" upper="3.14159" effort="78" velocity="0.52" />
       <origin rpy="-0.00000 0.00000 0.00000" xyz="0.10000 0.00000 0.09400" />
-      <parent link="${prefix}${parent}" />
-      <child link="${prefix}${name}" />
+      <parent link="${tf_prefix}${parent}" />
+      <child link="${tf_prefix}${name}" />
       <axis xyz="0 1 0" />
     </joint>
-    <link name="${prefix}${name}">
-      <collision name="${prefix}${name}_collision">
+    <link name="${tf_prefix}${name}">
+      <collision name="${tf_prefix}${name}_collision">
         <origin rpy="0.00000 0.00000 0.00000" xyz="0.00000 0.00000 0.00000" />
         <geometry>
@@ -26,5 +26,5 @@
         <mass value="1.58688811563124" />
       </inertial>
-      <visual name="${prefix}${name}_visual">
+      <visual name="${tf_prefix}${name}_visual">
         <origin rpy="0.00000 -0.00000 -0.00000" xyz="0.00000 0.00000 0.00000" />
         <geometry>
@@ -34,6 +34,7 @@
       </visual>
     </link>
-    <xacro:joint_hardware joint_name="${prefix}${name}_joint" hardware="${hardware}" p="1000000" d="0.5"/>
-    <xacro:rbs_materials link_name="${prefix}${name}" link_type="main_link" />
+    <xacro:joint_hardware joint_name="${tf_prefix}${name}_joint" hardware="${hardware}"
+      p="100000" d="0.2" />
+    <xacro:rbs_materials link_name="${tf_prefix}${name}" link_type="main_link" />
   </xacro:macro>
 </robot>

File: urdf/rbs_arm.xacro (robot description, xacro)
@@ -4,11 +4,11 @@
     <xacro:arg name="hardware" default="fake" />
     <xacro:arg name="simulation_controllers" default="" />
-    <xacro:arg name="prefix" default="" />
+    <xacro:arg name="tf_prefix" default="" />
     <xacro:property name="hardware" default="$(arg hardware)" />
-    <xacro:property name="prefix" default="$(arg prefix)" />
+    <xacro:property name="tf_prefix" default="$(arg tf_prefix)" />
     <xacro:include filename="$(find rbs_arm)/urdf/rbs_arm_macro.xacro" />
     <link name="world" />
     <!-- ROBOT-->
-    <xacro:rbs_arm parent="world" hardware="$(arg hardware)" prefix="$(arg prefix)">
+    <xacro:rbs_arm parent="world" hardware="$(arg hardware)" tf_prefix="$(arg tf_prefix)">
         <origin xyz="0.0 0.0 0.0" rpy="0.0 0.0 0.0" />
     </xacro:rbs_arm>
@@ -20,5 +20,5 @@
                 name="ign_ros2_control::IgnitionROS2ControlPlugin">
                 <parameters>$(arg simulation_controllers)</parameters>
-                <controller_manager_node_name>${prefix}/controller_manager</controller_manager_node_name>
+                <controller_manager_node_name>${tf_prefix}/controller_manager</controller_manager_node_name>
             </plugin>
         </gazebo>
