Commit message: prefix to tf prefix and rework launch files

File: urdf/rbs_arm_macro.xacro (robot description, xacro)
@@ -3,64 +3,64 @@
   <xacro:include filename="$(find rbs_arm)/urdf/rbs_arm_ros2_control.xacro" />
   <xacro:include filename="$(find rbs_arm)/urdf/inc/materials.xacro" />
-  <xacro:macro name="rbs_arm" params="prefix *origin parent hardware">
+  <xacro:macro name="rbs_arm" params="tf_prefix *origin parent hardware">
     <!-- ros2_control description macros-->
-    <xacro:rbs_arm_ros2_control name="rbs_arm_hardware_interface" prefix="${prefix}"
+    <xacro:rbs_arm_ros2_control name="rbs_arm_hardware_interface" tf_prefix="${tf_prefix}"
       hardware="${hardware}" />
     <!-- JOINTS-->
-    <joint name="${prefix}base_link_joint" type="fixed">
+    <joint name="${tf_prefix}base_link_joint" type="fixed">
       <xacro:insert_block name="origin" />
       <parent link="${parent}" />
-      <child link="${prefix}base_link" />
-    </joint>
-    <joint name="${prefix}ee_link_joint" type="revolute">
+      <child link="${tf_prefix}base_link" />
+    </joint>
+    <joint name="${tf_prefix}ee_link_joint" type="revolute">
       <limit lower="-1.5708" upper="3.14159" effort="78" velocity="0.52" />
       <origin rpy="0.00000 0.00000 0.00000" xyz="0.10000 0.00000 0.09473" />
-      <parent link="${prefix}fork.003_link" />
-      <child link="${prefix}ee_link" />
+      <parent link="${tf_prefix}fork.003_link" />
+      <child link="${tf_prefix}ee_link" />
       <axis xyz="0 1 0" />
     </joint>
-    <joint name="${prefix}fork002_link_joint" type="revolute">
+    <joint name="${tf_prefix}fork002_link_joint" type="revolute">
       <limit lower="-3.14159" upper="3.14159" effort="78" velocity="0.52" />
       <origin rpy="0.00000 0.00000 0.00000" xyz="0.00000 0.00000 0.13300" />
-      <parent link="${prefix}main_link" />
-      <child link="${prefix}fork.002_link" />
+      <parent link="${tf_prefix}main_link" />
+      <child link="${tf_prefix}fork.002_link" />
       <axis xyz="0 0 1" />
     </joint>
-    <joint name="${prefix}fork003_link_joint" type="revolute">
+    <joint name="${tf_prefix}fork003_link_joint" type="revolute">
       <limit lower="-3.14159" upper="3.14159" effort="78" velocity="0.52" />
       <origin rpy="0.00000 0.00000 0.00000" xyz="0.00000 0.00000 0.13300" />
-      <parent link="${prefix}main.001_link" />
-      <child link="${prefix}fork.003_link" />
+      <parent link="${tf_prefix}main.001_link" />
+      <child link="${tf_prefix}fork.003_link" />
       <axis xyz="0 0 1" />
     </joint>
-    <joint name="${prefix}fork001_link_joint" type="revolute">
+    <joint name="${tf_prefix}fork001_link_joint" type="revolute">
       <limit lower="-3.14159" upper="3.14159" effort="78" velocity="0.52" />
       <origin rpy="0.00000 0.00000 -0.00000" xyz="0.00000 -0.00000 0.17833" />
-      <parent link="${prefix}base_link" />
-      <child link="${prefix}fork_link" />
+      <parent link="${tf_prefix}base_link" />
+      <child link="${tf_prefix}fork_link" />
       <axis xyz="0 0 1" />
     </joint>
-    <joint name="${prefix}main002_link_joint" type="revolute">
+    <joint name="${tf_prefix}main002_link_joint" type="revolute">
       <limit lower="-1.5708" upper="3.14159" effort="78" velocity="0.52" />
       <origin rpy="-0.00000 0.00000 0.00000" xyz="0.10000 0.00000 0.09400" />
-      <parent link="${prefix}fork.002_link" />
-      <child link="${prefix}main.001_link" />
+      <parent link="${tf_prefix}fork.002_link" />
+      <child link="${tf_prefix}main.001_link" />
       <axis xyz="0 1 0" />
     </joint>
-    <joint name="${prefix}main001_link_joint" type="revolute">
+    <joint name="${tf_prefix}main001_link_joint" type="revolute">
       <limit lower="-1.5708" upper="3.14159" effort="78" velocity="0.52" />
       <origin rpy="0.00000 0.00000 0.00000" xyz="0.10000 0.00000 0.09400" />
-      <parent link="${prefix}fork_link" />
-      <child link="${prefix}main_link" />
+      <parent link="${tf_prefix}fork_link" />
+      <child link="${tf_prefix}main_link" />
       <axis xyz="0 1 0" />
     </joint>
-    <joint name="${prefix}tool0_joint" type="fixed">
+    <joint name="${tf_prefix}tool0_joint" type="fixed">
       <origin rpy="-0.00000 0.00000 -0.00000" xyz="0.00001 -0.00010 0.11000" />
-      <parent link="${prefix}ee_link" />
-      <child link="${prefix}tool0" />
+      <parent link="${tf_prefix}ee_link" />
+      <child link="${tf_prefix}tool0" />
     </joint>
     <!-- LINKS-->
-    <link name="${prefix}base_link">
-      <collision name="${prefix}base_collision">
+    <link name="${tf_prefix}base_link">
+      <collision name="${tf_prefix}base_collision">
         <origin rpy="0.00000 0.00000 0.00000" xyz="0.00000 0.00000 0.00000" />
         <geometry>
@@ -76,5 +76,5 @@
         <mass value="1.88031044620482" />
       </inertial>
-      <visual name="${prefix}base_visual">
+      <visual name="${tf_prefix}base_visual">
         <origin rpy="0.00000 0.00000 0.00000" xyz="0.00000 0.00000 0.00000" />
         <geometry>
@@ -84,6 +84,6 @@
       </visual>
     </link>
-    <link name="${prefix}ee_link">
-      <collision name="${prefix}ee_collision">
+    <link name="${tf_prefix}ee_link">
+      <collision name="${tf_prefix}ee_collision">
         <origin rpy="-0.00000 0.00000 -0.00000" xyz="0.00000 -0.00000 0.00000" />
         <geometry>
@@ -99,5 +99,5 @@
         <mass value="1.88031044620482" />
       </inertial>
-      <visual name="${prefix}ee_visual">
+      <visual name="${tf_prefix}ee_visual">
         <origin rpy="0.00000 0.00000 0.00000" xyz="0.00000 -0.00000 0.00000" />
         <geometry>
@@ -107,6 +107,6 @@
       </visual>
     </link>
-    <link name="${prefix}fork.002_link">
-      <collision name="${prefix}fork.002_collision">
+    <link name="${tf_prefix}fork.002_link">
+      <collision name="${tf_prefix}fork.002_collision">
         <origin rpy="0.00000 0.00000 0.00000" xyz="0.00000 -0.00000 0.00000" />
         <geometry>
@@ -122,5 +122,5 @@
         <mass value="1.12472202892859" />
       </inertial>
-      <visual name="${prefix}fork.002_visual">
+      <visual name="${tf_prefix}fork.002_visual">
         <origin rpy="0.00000 -0.00000 -0.00000" xyz="0.00000 -0.00000 0.00000" />
         <geometry>
@@ -130,6 +130,6 @@
       </visual>
     </link>
-    <link name="${prefix}fork.003_link">
-      <collision name="${prefix}fork.003_collision">
+    <link name="${tf_prefix}fork.003_link">
+      <collision name="${tf_prefix}fork.003_collision">
         <origin rpy="-0.00000 0.00000 0.00000" xyz="0.00000 -0.00000 0.00000" />
         <geometry>
@@ -145,5 +145,5 @@
         <mass value="1.12472202892859" />
       </inertial>
-      <visual name="${prefix}fork.003_visual">
+      <visual name="${tf_prefix}fork.003_visual">
         <origin rpy="-0.00000 0.00000 -0.00000" xyz="0.00000 -0.00000 0.00000" />
         <geometry>
@@ -153,6 +153,6 @@
       </visual>
     </link>
-    <link name="${prefix}fork_link">
-      <collision name="${prefix}fork_collision">
+    <link name="${tf_prefix}fork_link">
+      <collision name="${tf_prefix}fork_collision">
         <origin rpy="0.00000 0.00000 0.00000" xyz="-0.00000 0.00000 0.00000" />
         <geometry>
@@ -168,5 +168,5 @@
         <mass value="1.12472202892859" />
       </inertial>
-      <visual name="${prefix}fork_visual">
+      <visual name="${tf_prefix}fork_visual">
         <origin rpy="0.00000 0.00000 -0.00000" xyz="-0.00000 0.00000 0.00000" />
         <geometry>
@@ -176,6 +176,6 @@
       </visual>
     </link>
-    <link name="${prefix}main.001_link">
-      <collision name="${prefix}main.001_collision">
+    <link name="${tf_prefix}main.001_link">
+      <collision name="${tf_prefix}main.001_collision">
         <origin rpy="0.00000 0.00000 0.00000" xyz="0.00000 0.00000 0.00000" />
         <geometry>
@@ -191,5 +191,5 @@
         <mass value="1.58688811563124" />
       </inertial>
-      <visual name="${prefix}main.001_visual">
+      <visual name="${tf_prefix}main.001_visual">
         <origin rpy="0.00000 -0.00000 -0.00000" xyz="0.00000 0.00000 0.00000" />
         <geometry>
@@ -199,6 +199,6 @@
       </visual>
     </link>
-    <link name="${prefix}main_link">
-      <collision name="${prefix}main_collision">
+    <link name="${tf_prefix}main_link">
+      <collision name="${tf_prefix}main_collision">
         <origin rpy="0.00000 0.00000 0.00000" xyz="0.00000 0.00000 0.00000" />
         <geometry>
@@ -214,5 +214,5 @@
         <mass value="1.58688811563124" />
       </inertial>
-      <visual name="${prefix}main_visual">
+      <visual name="${tf_prefix}main_visual">
         <origin rpy="0.00000 -0.00000 -0.00000" xyz="0.00000 0.00000 0.00000" />
         <geometry>
@@ -222,7 +222,7 @@
       </visual>
     </link>
-    <link name="${prefix}tool0" />
+    <link name="${tf_prefix}tool0" />
     <!-- MATERIALS-->
-    <xacro:rbs_materials link_name="${prefix}main_link" link_type="main_link" />
+    <xacro:rbs_materials link_name="${tf_prefix}main_link" link_type="main_link" />
   </xacro:macro>
 </robot>

File: urdf/rbs_arm_modular.xacro (robot description, xacro)
@@ -4,8 +4,11 @@
   <xacro:arg name="hardware" default="gazebo" />
   <xacro:arg name="simulation_controllers" default="" />
-  <xacro:arg name="prefix" default="" />
+  <xacro:arg name="tf_prefix" default="" />
+  <xacro:arg name="namespace" default="arm0"/>
   <xacro:include filename="$(find rbs_arm)/urdf/rbs_arm_modular_macro.xacro" />
   <link name="world" />
-  <xacro:rbs_arm parent="world" prefix="$(arg prefix)" hardware="$(arg hardware)"
-    gripper_name="$(arg gripper_name)" controllers="$(arg simulation_controllers)" />
+  <xacro:rbs_arm namespace="$(arg namespace)" parent="world" tf_prefix="$(arg tf_prefix)" hardware="$(arg hardware)"
+    gripper_name="$(arg gripper_name)" controllers="$(arg simulation_controllers)">
+    <origin xyz="0 0 0" rpy="0 0 0" />
+  </xacro:rbs_arm>
 </robot>

File: urdf/rbs_arm_modular_macro.xacro (robot description, xacro)
@@ -1,40 +1,45 @@
 <?xml version="1.0" encoding="UTF-8"?>
 <robot xmlns:xacro="http://www.ros.org/wiki/xacro">
- <xacro:macro name="rbs_arm" params="parent prefix hardware gripper_name controllers">
-  <xacro:include filename="$(find rbs_arm)/urdf/inc/rbs_base_link.xacro" />
-  <xacro:include filename="$(find rbs_arm)/urdf/inc/rbs_ee_link.xacro" />
-  <xacro:include filename="$(find rbs_arm)/urdf/inc/rbs_fork_link.xacro" />
-  <xacro:include filename="$(find rbs_arm)/urdf/inc/rbs_main_link.xacro" />
-  <!-- origin to define robot position in the world-->
-  <xacro:base_link parent="${parent}" prefix="${prefix}" hardware="${hardware}">
-    <origin xyz="0 0 0" rpy="0 0 0" />
-  </xacro:base_link>
-  <xacro:fork_link parent="base_link"  name="fork0_link" prefix="${prefix}" hardware="${hardware}" />
-  <xacro:main_link parent="fork0_link" name="main0_link" prefix="${prefix}" hardware="${hardware}" />
-  <xacro:fork_link parent="main0_link" name="fork1_link" prefix="${prefix}" hardware="${hardware}" />
-  <xacro:main_link parent="fork1_link" name="main1_link" prefix="${prefix}" hardware="${hardware}" />
-  <xacro:fork_link parent="main1_link" name="fork2_link" prefix="${prefix}" hardware="${hardware}" />
-  <!-- ee link also contain tool0-->
-  <xacro:ee_link parent="fork2_link" prefix="${prefix}" hardware="${hardware}" />
-  <xacro:if value="${gripper_name=='rbs_gripper'}">
-    <xacro:include filename="$(find rbs_gripper)/urdf/rbs_gripper_macro.xacro" />
-    <xacro:rbs_gripper prefix="${prefix}" gripper_name="rbs_gripper" parent="tool0"
-      hardware="${hardware}">
-      <origin xyz="0.0 0.0 0.0" rpy="0.0 0.0 0.0" />
-    </xacro:rbs_gripper>
-  </xacro:if>
-  <xacro:if value="${hardware=='gazebo'}">
-    <gazebo>
-      <plugin filename="libign_ros2_control-system.so"
-        name="ign_ros2_control::IgnitionROS2ControlPlugin">
-        <parameters>$(arg simulation_controllers)</parameters>
-        <controller_manager_node_name>${prefix}/controller_manager</controller_manager_node_name>
+  <xacro:macro name="rbs_arm" params="namespace parent *origin tf_prefix hardware gripper_name controllers">
+    <xacro:include filename="$(find rbs_arm)/urdf/inc/rbs_base_link.xacro" />
+    <xacro:include filename="$(find rbs_arm)/urdf/inc/rbs_ee_link.xacro" />
+    <xacro:include filename="$(find rbs_arm)/urdf/inc/rbs_fork_link.xacro" />
+    <xacro:include filename="$(find rbs_arm)/urdf/inc/rbs_main_link.xacro" />
+    <!-- BEGIN robot description  -->
+    <xacro:base_link parent="${parent}" tf_prefix="${tf_prefix}" hardware="${hardware}">
+      <xacro:insert_block name="origin" />
+    </xacro:base_link>
+    <xacro:fork_link parent="base_link"  name="fork0_link" tf_prefix="${tf_prefix}" hardware="${hardware}" />
+    <xacro:main_link parent="fork0_link" name="main0_link" tf_prefix="${tf_prefix}" hardware="${hardware}" />
+    <xacro:fork_link parent="main0_link" name="fork1_link" tf_prefix="${tf_prefix}" hardware="${hardware}" />
+    <xacro:main_link parent="fork1_link" name="main1_link" tf_prefix="${tf_prefix}" hardware="${hardware}" />
+    <xacro:fork_link parent="main1_link" name="fork2_link" tf_prefix="${tf_prefix}" hardware="${hardware}" />
+    <!-- ee link also contain tool0-->
+    <xacro:ee_link parent="fork2_link" tf_prefix="${tf_prefix}" hardware="${hardware}" />
+    <!-- END robot description -->
+    <!-- Insert gripper in robot description if exist -->
+    <xacro:if value="${gripper_name=='rbs_gripper'}">
+      <xacro:include filename="$(find rbs_gripper)/urdf/rbs_gripper_macro.xacro" />
+      <xacro:rbs_gripper tf_prefix="${tf_prefix}" gripper_name="rbs_gripper" parent="${tf_prefix}tool0"
+        hardware="${hardware}">
+        <origin xyz="0.0 0.0 0.0" rpy="0.0 0.0 0.0" />
+      </xacro:rbs_gripper>
+    </xacro:if>
+    <!-- If hardware == gazebo so insert additional parameters for it -->
+    <xacro:if value="${hardware=='gazebo'}">
+      <gazebo>
+        <plugin filename="libign_ros2_control-system.so"
+          name="ign_ros2_control::IgnitionROS2ControlPlugin">
+          <parameters>$(arg simulation_controllers)</parameters>
+          <!-- <controller_manager_prefix_node_name>${namespace}</controller_manager_prefix_node_name> -->
+          <!-- <controller_manager_node_name>/${namespace}/controller_manager</controller_manager_node_name> -->
           <ros>
-            <remapping>/motion_controller_handle/target_frame:=/target_frame</remapping>
-            <remapping>/cartesian_motion_controller/target_frame:=/target_frame</remapping>
+            <namespace>${namespace}</namespace>
+            <!-- <remapping>/motion_controller_handle/target_frame:=/target_frame</remapping> -->
+            <!-- <remapping>/cartesian_motion_controller/target_frame:=/target_frame</remapping> -->
           </ros>
-      </plugin>
-    </gazebo>
-  </xacro:if>
- </xacro:macro>
+        </plugin>
+      </gazebo>
+    </xacro:if>
+  </xacro:macro>
 </robot>

File: urdf/rbs_arm_ros2_control.xacro (robot description, xacro)
@@ -2,5 +2,5 @@
 <robot xmlns:xacro="http://www.ros.org/wiki/xacro">
     <xacro:include filename="$(find rbs_arm)/urdf/inc/joint_interface.xacro" />
-    <xacro:macro name="rbs_arm_ros2_control" params="name hardware prefix">
+    <xacro:macro name="rbs_arm_ros2_control" params="name hardware tf_prefix">
         <ros2_control name="${name}" type="system">
             <hardware>
@@ -12,10 +12,10 @@
                 </xacro:if>
             </hardware>
-            <xacro:joint_interface name="${prefix}fork001_link_joint" p="1000" d="0.5" />
-            <xacro:joint_interface name="${prefix}main001_link_joint" p="1000" d="0.5" />
-            <xacro:joint_interface name="${prefix}fork002_link_joint" p="500" d="0.5" />
-            <xacro:joint_interface name="${prefix}main002_link_joint" p="100" d="0.5" />
-            <xacro:joint_interface name="${prefix}fork003_link_joint" p="10" d="0.5" />
-            <xacro:joint_interface name="${prefix}ee_link_joint" p="10" d="0.5" />
+            <xacro:joint_interface name="${tf_prefix}fork001_link_joint" p="1000" d="0.5" />
+            <xacro:joint_interface name="${tf_prefix}main001_link_joint" p="1000" d="0.5" />
+            <xacro:joint_interface name="${tf_prefix}fork002_link_joint" p="500" d="0.5" />
+            <xacro:joint_interface name="${tf_prefix}main002_link_joint" p="100" d="0.5" />
+            <xacro:joint_interface name="${tf_prefix}fork003_link_joint" p="10" d="0.5" />
+            <xacro:joint_interface name="${tf_prefix}ee_link_joint" p="10" d="0.5" />
         </ros2_control>
     </xacro:macro>

File: urdf/sensors.xacro (robot description, xacro)
@@ -1,6 +1,6 @@
 <?xml version="1.0"?>
 <robot xmlns:xacro="http://www.ros.org/wiki/xacro" name="rack">
-    <xacro:macro name="rgbd" params="*origin parent prefix">
-        <link name="${prefix}rgbd_camera">
+    <xacro:macro name="rgbd" params="*origin parent tf_prefix">
+        <link name="${tf_prefix}rgbd_camera">
             <inertial>
                 <origin xyz="0.0 0.0 0.0" rpy="0.0 0.0 0.0"/>
@@ -25,6 +25,6 @@
             </collision>
         </link>
-        <gazebo reference = "${prefix}rgbd_camera">
-            <sensor name="${prefix}rgbd_camera" type="rgbd_camera">
+        <gazebo reference = "${tf_prefix}rgbd_camera">
+            <sensor name="${tf_prefix}rgbd_camera" type="rgbd_camera">
                 <camera>
                     <horizontal_fov>1.047</horizontal_fov>
@@ -41,20 +41,20 @@
                 <update_rate>30</update_rate>
                 <visualize>true</visualize>
-                <topic>${prefix}rgbd_camera</topic>
+                <topic>${tf_prefix}rgbd_camera</topic>
                 <enable_metrics>true</enable_metrics>
             </sensor>
         </gazebo>
-        <joint name="${prefix}rgbd_camera_to_parent" type="fixed">
+        <joint name="${tf_prefix}rgbd_camera_to_parent" type="fixed">
             <parent link="${parent}" />
-            <child link="${prefix}rgbd_camera" />
+            <child link="${tf_prefix}rgbd_camera" />
             <xacro:insert_block name="origin" />
         </joint>
     </xacro:macro>
-    <xacro:macro name="rbs_fts" params="name prefix link">
-    <ros2_control name="${prefix}${name}" type="sensor">
+    <xacro:macro name="rbs_fts" params="name tf_prefix link">
+    <ros2_control name="${tf_prefix}${name}" type="sensor">
       <hardware>
           <plugin>ign_ros2_control/IgnitionFts</plugin>
       </hardware>
-      <sensor name="${prefix}${name}">
+      <sensor name="${tf_prefix}${name}">
         <state_interface name="force.x"/>
         <state_interface name="force.y"/>
@@ -65,6 +65,6 @@
       </sensor>
     </ros2_control>
-    <gazebo reference="${prefix}${link}_joint">
-        <sensor name="${prefix}${name}" type="force_torque">
+    <gazebo reference="${tf_prefix}${link}_joint">
+        <sensor name="${tf_prefix}${name}" type="force_torque">
           <always_on>true</always_on>
           <update_rate>50</update_rate>
