Commit message: add simple moveit and ros2-control config generation

File: scripts/robot_6_dof.urdf (robot description, URDF)
Before this commit: robot rbs_arm, 8 links, 7 joints
Links:
- added link rbs_arm_link_tool0
Joints:
- added joint rbs_arm_joint_tool0: type fixed, parent rbs_arm_link_6, child rbs_arm_tool0, origin xyz=0 0 0.11 rpy=0 0 0
