Commit message: add urdf generation via odio_urdf

File: urdf/inc/rbs_ee_link.xacro (robot description, xacro)
@@ -21,5 +21,5 @@
         <origin rpy="-0.00000 0.00000 -0.00000" xyz="0.00000 -0.00000 0.00000" />
         <geometry>
-          <mesh filename="file://$(find rbs_arm)/meshes/collision/tail_link.stl"
+          <mesh filename="file://$(find rbs_arm)/meshes/collision/ee_link.stl"
             scale="1.00000 1.00000 1.00000" />
         </geometry>
@@ -35,5 +35,5 @@
         <origin rpy="0.00000 0.00000 0.00000" xyz="0.00000 -0.00000 0.00000" />
         <geometry>
-          <mesh filename="file://$(find rbs_arm)/meshes/visual/tail_link.dae"
+          <mesh filename="file://$(find rbs_arm)/meshes/visual/ee_link.dae"
             scale="1.00000 1.00000 1.00000" />
         </geometry>

File: urdf/inc/rbs_fork_link.xacro (robot description, xacro)
@@ -4,5 +4,5 @@
     <xacro:include filename="$(find rbs_arm)/urdf/inc/joint_hardware.xacro" />
     <xacro:include filename="$(find rbs_arm)/urdf/inc/materials.xacro" />
-    <joint name="${tf_prefix}${name}_joint" type="continuous">
+    <joint name="${tf_prefix}${name}_joint" type="revolute">
       <limit lower="-3.14159" upper="3.14159" effort="78" velocity="0.52" />
       <xacro:if value="${parent=='base_link'}">
@@ -20,5 +20,5 @@
         <origin rpy="0.00000 0.00000 0.00000" xyz="0.00000 -0.00000 0.00000" />
         <geometry>
-          <mesh filename="file://$(find rbs_arm)/meshes/collision/fork.stl"
+          <mesh filename="file://$(find rbs_arm)/meshes/collision/fork_link.stl"
             scale="1.00000 1.00000 1.00000" />
         </geometry>
@@ -34,5 +34,5 @@
         <origin rpy="0.00000 -0.00000 -0.00000" xyz="0.00000 -0.00000 0.00000" />
         <geometry>
-          <mesh filename="file://$(find rbs_arm)/meshes/visual/fork.dae"
+          <mesh filename="file://$(find rbs_arm)/meshes/visual/fork_link.dae"
             scale="1.00000 1.00000 1.00000" />
         </geometry>

File: urdf/rbs_arm_modular_macro.xacro (robot description, xacro)
@@ -32,10 +32,6 @@
           name="ign_ros2_control::IgnitionROS2ControlPlugin">
           <parameters>$(arg simulation_controllers)</parameters>
-          <!-- <controller_manager_prefix_node_name>${namespace}</controller_manager_prefix_node_name> -->
-          <!-- <controller_manager_node_name>/${namespace}/controller_manager</controller_manager_node_name> -->
           <ros>
             <namespace>${namespace}</namespace>
-            <!-- <remapping>/motion_controller_handle/target_frame:=/target_frame</remapping> -->
-            <!-- <remapping>/cartesian_motion_controller/target_frame:=/target_frame</remapping> -->
           </ros>
         </plugin>

Commit message: update for compatibility with rbs framework

File: urdf/inc/rbs_ee_link.xacro (robot description, xacro)
@@ -12,4 +12,5 @@
     </joint>
     <joint name="${tf_prefix}tool0_joint" type="fixed">
+      <!-- <limit lower="0.00000" upper="0.00000" effort="0.00000" velocity="0.00000" /> -->
       <origin rpy="0.00000 0.00000 0.00000" xyz="0.00000 0.00000 0.11000" />
       <parent link="${tf_prefix}ee_link" />

File: urdf/rbs_arm_modular.xacro (robot description, xacro)
@@ -6,9 +6,15 @@
   <xacro:arg name="tf_prefix" default="" />
   <xacro:arg name="namespace" default="arm0"/>
+  <xacro:arg name="x" default="0.0" />
+  <xacro:arg name="y" default="0.0" />
+  <xacro:arg name="z" default="0.0" />
+  <xacro:arg name="roll" default="0.0" />
+  <xacro:arg name="pitch" default="0.0" />
+  <xacro:arg name="yaw" default="0.0" />
   <xacro:include filename="$(find rbs_arm)/urdf/rbs_arm_modular_macro.xacro" />
   <link name="world" />
   <xacro:rbs_arm namespace="$(arg namespace)" parent="world" tf_prefix="$(arg tf_prefix)" hardware="$(arg hardware)"
     gripper_name="$(arg gripper_name)" controllers="$(arg simulation_controllers)">
-    <origin xyz="0 0 0" rpy="0 0 0" />
+    <origin xyz="$(arg x) $(arg y) $(arg z)" rpy="$(arg roll) $(arg pitch) $(arg yaw)" />
   </xacro:rbs_arm>
 </robot>

File: urdf/rbs_arm_modular_macro.xacro (robot description, xacro)
@@ -6,4 +6,5 @@
     <xacro:include filename="$(find rbs_arm)/urdf/inc/rbs_fork_link.xacro" />
     <xacro:include filename="$(find rbs_arm)/urdf/inc/rbs_main_link.xacro" />
+    <xacro:include filename="$(find rbs_arm)/urdf/sensors.xacro"/>
     <!-- BEGIN robot description  -->
     <xacro:base_link parent="${parent}" tf_prefix="${tf_prefix}" hardware="${hardware}">
@@ -28,4 +29,5 @@
     <!-- If hardware == gazebo so insert additional parameters for it -->
     <xacro:if value="${hardware=='gazebo'}">
+      <xacro:rbs_fts name="fts_sensor" tf_prefix="${tf_prefix}" link="${tf_prefix}tool0"/>
       <gazebo>
         <plugin filename="libign_ros2_control-system.so"

File: urdf/sensors.xacro (robot description, xacro)
@@ -66,12 +66,13 @@
     </ros2_control>
     <gazebo reference="${tf_prefix}${link}_joint">
+        <preserveFixedJoint>true</preserveFixedJoint>
         <sensor name="${tf_prefix}${name}" type="force_torque">
           <always_on>true</always_on>
           <update_rate>50</update_rate>
           <visualize>true</visualize>
-          <topic>ft_data</topic>
+          <topic>${tf_prefix}ft_data</topic>
           <force_torque>
             <frame>sensor</frame>
-            <measure_direction>parent_to_child</measure_direction>
+            <measure_direction>child_to_parent</measure_direction>
           </force_torque>
         </sensor>
