Commit message: add different pd joint gains

File: urdf/inc/joint_interface.xacro (robot description, xacro)
@@ -16,4 +16,5 @@
                         <!-- <param name="p">${p}</param> -->
                         <!-- <param name="d">${d}</param> -->
+                        <!-- <command_interface name="effort"/> -->
                         <state_interface name="position"/>
                         <state_interface name="velocity"/>

File: urdf/inc/materials.xacro (robot description, xacro)
@@ -3,4 +3,12 @@
   <xacro:macro name="rbs_materials" params="link_name link_type">
     <gazebo reference="${link_name}">
+      <soft_contact>
+        <dart>
+          <bone_attachment>100</bone_attachment>
+          <stiffness>100</stiffness>
+          <damping>10</damping>
+          <flesh_mass_fraction>0.050000000000000003</flesh_mass_fraction>
+        </dart>
+      </soft_contact>
       <visual>
         <material>

File: urdf/inc/rbs_ee_link.xacro (robot description, xacro)
@@ -1,5 +1,5 @@
 <?xml version="1.0" encoding="UTF-8"?>
 <robot xmlns:xacro="http://www.ros.org/wiki/xacro">
-  <xacro:macro name="ee_link" params="tf_prefix parent hardware">
+  <xacro:macro name="ee_link" params="tf_prefix parent hardware p d">
     <xacro:include filename="$(find rbs_arm)/urdf/inc/joint_hardware.xacro" />
     <xacro:include filename="$(find rbs_arm)/urdf/inc/materials.xacro" />
@@ -12,5 +12,4 @@
     </joint>
     <joint name="${tf_prefix}tool0_joint" type="fixed">
-      <!-- <limit lower="0.00000" upper="0.00000" effort="0.00000" velocity="0.00000" /> -->
       <origin rpy="0.00000 0.00000 0.00000" xyz="0.00000 0.00000 0.11000" />
       <parent link="${tf_prefix}ee_link" />
@@ -41,5 +40,5 @@
       </visual>
     </link>
-    <xacro:joint_hardware joint_name="${tf_prefix}ee_link_joint" hardware="${hardware}" p="10" d="0.5" />
+    <xacro:joint_hardware joint_name="${tf_prefix}ee_link_joint" hardware="${hardware}" p="${p}" d="${d}" />
     <xacro:rbs_materials link_name="${tf_prefix}ee_link" link_type="ee_link" />
   </xacro:macro>

File: urdf/inc/rbs_fork_link.xacro (robot description, xacro)
@@ -1,5 +1,5 @@
 <?xml version="1.0" encoding="UTF-8"?>
 <robot xmlns:xacro="http://www.ros.org/wiki/xacro">
-  <xacro:macro name="fork_link" params="tf_prefix parent name hardware">
+  <xacro:macro name="fork_link" params="tf_prefix parent name hardware p d">
     <xacro:include filename="$(find rbs_arm)/urdf/inc/joint_hardware.xacro" />
     <xacro:include filename="$(find rbs_arm)/urdf/inc/materials.xacro" />
@@ -39,5 +39,5 @@
       </visual>
     </link>
-    <xacro:joint_hardware joint_name="${tf_prefix}${name}_joint" hardware="${hardware}" p="1000000" d="0.5" />
+    <xacro:joint_hardware joint_name="${tf_prefix}${name}_joint" hardware="${hardware}" p="${p}" d="${d}" />
     <xacro:rbs_materials link_name="${tf_prefix}${name}" link_type="fork" />
   </xacro:macro>

File: urdf/inc/rbs_main_link.xacro (robot description, xacro)
@@ -1,5 +1,5 @@
 <?xml version="1.0" encoding="UTF-8"?>
 <robot xmlns:xacro="http://www.ros.org/wiki/xacro">
-  <xacro:macro name="main_link" params="tf_prefix parent name hardware">
+  <xacro:macro name="main_link" params="tf_prefix parent name hardware p d">
     <xacro:include filename="$(find rbs_arm)/urdf/inc/joint_hardware.xacro" />
     <xacro:include filename="$(find rbs_arm)/urdf/inc/materials.xacro" />
@@ -35,5 +35,5 @@
     </link>
     <xacro:joint_hardware joint_name="${tf_prefix}${name}_joint" hardware="${hardware}"
-      p="100000" d="0.2" />
+      p="${p}" d="${d}" />
     <xacro:rbs_materials link_name="${tf_prefix}${name}" link_type="main_link" />
   </xacro:macro>

File: urdf/rbs_arm_modular_macro.xacro (robot description, xacro)
@@ -11,11 +11,17 @@
       <xacro:insert_block name="origin" />
     </xacro:base_link>
-    <xacro:fork_link parent="base_link"  name="fork0_link" tf_prefix="${tf_prefix}" hardware="${hardware}" />
-    <xacro:main_link parent="fork0_link" name="main0_link" tf_prefix="${tf_prefix}" hardware="${hardware}" />
-    <xacro:fork_link parent="main0_link" name="fork1_link" tf_prefix="${tf_prefix}" hardware="${hardware}" />
-    <xacro:main_link parent="fork1_link" name="main1_link" tf_prefix="${tf_prefix}" hardware="${hardware}" />
-    <xacro:fork_link parent="main1_link" name="fork2_link" tf_prefix="${tf_prefix}" hardware="${hardware}" />
+    <xacro:fork_link parent="base_link"  name="fork0_link" tf_prefix="${tf_prefix}" hardware="${hardware}"
+      p="10000" d="0.2"  />
+    <xacro:main_link parent="fork0_link" name="main0_link" tf_prefix="${tf_prefix}" hardware="${hardware}"
+      p="10000" d="0.2"/>
+    <xacro:fork_link parent="main0_link" name="fork1_link" tf_prefix="${tf_prefix}" hardware="${hardware}"
+      p="10000" d="0.2"/>
+    <xacro:main_link parent="fork1_link" name="main1_link" tf_prefix="${tf_prefix}" hardware="${hardware}"
+      p="1000" d="0.2"/>
+    <xacro:fork_link parent="main1_link" name="fork2_link" tf_prefix="${tf_prefix}" hardware="${hardware}"
+      p="100" d="0.2"/>
     <!-- ee link also contain tool0-->
-    <xacro:ee_link parent="fork2_link" tf_prefix="${tf_prefix}" hardware="${hardware}" />
+    <xacro:ee_link parent="fork2_link" tf_prefix="${tf_prefix}" hardware="${hardware}"
+      p="20" d="0.2"/>
     <!-- END robot description -->
     <!-- Insert gripper in robot description if exist -->
