Commit message: add test launch files for robot_builder module

File: urdf/inc/materials.xacro (robot description, xacro)
@@ -3,12 +3,4 @@
   <xacro:macro name="rbs_materials" params="link_name link_type">
     <gazebo reference="${link_name}">
-      <soft_contact>
-        <dart>
-          <bone_attachment>100</bone_attachment>
-          <stiffness>100</stiffness>
-          <damping>10</damping>
-          <flesh_mass_fraction>0.050000000000000003</flesh_mass_fraction>
-        </dart>
-      </soft_contact>
       <visual>
         <material>

File: urdf/inc/rbs_fork_link.xacro (robot description, xacro)
@@ -5,5 +5,5 @@
     <xacro:include filename="$(find rbs_arm)/urdf/inc/materials.xacro" />
     <joint name="${tf_prefix}${name}_joint" type="revolute">
-      <limit lower="-3.14159" upper="3.14159" effort="78" velocity="0.52" />
+      <limit lower="-6.14159" upper="6.14159" effort="78" velocity="0.52" />
       <xacro:if value="${parent=='base_link'}">
         <origin rpy="0.00000 0.00000 0.00000" xyz="0.00000 0.00000 0.17833" />
