Commit message: Migrate to new robot structure, refactor URDF, and update GazeboSim launch
- Transitioned to a new robot structure with updated URDF and Xacro definitions.
- Updated `rbs_ee_link.xacro`, `rbs_fork_link.xacro`, and `rbs_main_link.xacro`:
  - Adjusted joint limits, positions, and axes.
  - Standardized joint parameters and transformations.
  - Updated inertia, mass, and mesh references.
  - Added `initial_joint_position` for better initialization.
- Refactored `rbs_arm_modular_macro.xacro`:
  - Simplified link definitions and removed legacy gripper integration.
  - Improved Gazebo compatibility.
- Updated `sensors.xacro` to use `gz_ros2_control/GzFts` instead of `IgnitionFts`.
- Removed outdated URDF files (`rbs_arm.urdf`, `rbs_arm.xacro`, etc.).
- Refactored `display_gazebosim.launch.py`:
  - Introduced `OpaqueFunction` and `load_xacro_args` for improved launch setup.
  - Enhanced robot description processing using `xacro.process_file`.
  - Added a clock bridge node for time synchronization.
- Updated URDF/Xacro files:
  - Introduced `initial_joint_position` in `joint_hardware.xacro` and `joint_interface.xacro`.
  - Refactored `rbs_base_link.xacro` for improved formatting and efficiency.
- Modified collision and visual mesh files:
  - Added new STL files for individual axes and base link.
  - Removed outdated STL files (`ee_link.stl`, `fork_link.stl`, etc.).

File: urdf/inc/joint_hardware.xacro (robot description, xacro)
@@ -1,17 +1,19 @@
 <?xml version="1.0"?>
 <robot xmlns:xacro="http://www.ros.org/wiki/xacro">
-    <xacro:include filename="$(find rbs_arm)/urdf/inc/joint_interface.xacro" />
-    <xacro:macro name="joint_hardware" params="joint_name hardware p:=^ d:=^">
-        <ros2_control name="${joint_name}_hardware_interface" type="actuator">
-            <hardware>
-                <xacro:if value="${hardware=='gazebo'}">
-                    <plugin>gz_ros2_control/GazeboSimSystem</plugin>
-                </xacro:if>
-                <xacro:if value="${hardware=='mock'}">
-                    <plugin>mock_components/GenericSystem</plugin>
-                </xacro:if>
-            </hardware>
-            <xacro:joint_interface name="${joint_name}" p="${p}" d="${d}" />
-        </ros2_control>
-    </xacro:macro>
+  <xacro:include filename="$(find rbs_arm)/urdf/inc/joint_interface.xacro" />
+  <xacro:macro name="joint_hardware"
+    params="joint_name hardware p:=^ d:=^ initial_joint_position:=^|0.0">
+    <ros2_control name="${joint_name}_hardware_interface" type="actuator">
+      <hardware>
+        <xacro:if value="${hardware=='gazebo'}">
+          <plugin>gz_ros2_control/GazeboSimSystem</plugin>
+        </xacro:if>
+        <xacro:if value="${hardware=='mock'}">
+          <plugin>mock_components/GenericSystem</plugin>
+        </xacro:if>
+      </hardware>
+      <xacro:joint_interface name="${joint_name}" p="${p}" d="${d}"
+        initial_joint_position="${initial_joint_position}" />
+    </ros2_control>
+  </xacro:macro>
 </robot>

File: urdf/inc/joint_interface.xacro (robot description, xacro)
@@ -1,18 +1,20 @@
 <?xml version="1.0"?>
 <robot xmlns:xacro="http://www.ros.org/wiki/xacro">
-        <!-- Individual joint. -->
-  <xacro:macro name="joint_interface" params="name p:=^ d:=^">
-                <joint name="${name}">
-                        <command_interface name="position"/>
-                        <command_interface name="velocity"/>
-                        <!-- WARN When this active a robot falls down -->
-                        <!-- <command_interface name="effort"/> -->
-                        <param name="p">${p}</param>
-                        <param name="d">${d}</param>
-                        <!-- <command_interface name="effort"/> -->
-                        <state_interface name="position"/>
-                        <state_interface name="velocity"/>
-                        <!-- <state_interface name="acceleration"/> -->
-                </joint>
-        </xacro:macro>
+  <!-- Individual joint. -->
+  <xacro:macro name="joint_interface" params="name p:=^ d:=^ initial_joint_position:=^|0.0">
+    <joint name="${name}">
+      <command_interface name="position" />
+      <command_interface name="velocity" />
+      <!-- WARN When this active a robot falls down -->
+      <!-- <command_interface name="effort"/> -->
+      <param name="p">${p}</param>
+      <param name="d">${d}</param>
+      <!-- <command_interface name="effort"/> -->
+      <state_interface name="position">
+        <param name="initial_value">${initial_joint_position}</param>
+      </state_interface>
+      <state_interface name="velocity" />
+      <!-- <state_interface name="acceleration"/> -->
+    </joint>
+  </xacro:macro>
 </robot>

File: urdf/inc/rbs_base_link.xacro (robot description, xacro)
@@ -2,36 +2,35 @@
 <robot xmlns:xacro="http://www.ros.org/wiki/xacro">
   <xacro:macro name="base_link" params="parent tf_prefix *origin hardware">
-    <xacro:include filename="$(find rbs_arm)/urdf/inc/joint_hardware.xacro" />
-    <xacro:include filename="$(find rbs_arm)/urdf/inc/materials.xacro"/>
+    <xacro:include filename="$(find rbs_arm)/urdf/inc/joint_hardware.xacro"></xacro:include>
+    <xacro:include filename="$(find rbs_arm)/urdf/inc/materials.xacro"></xacro:include>
     <joint name="${tf_prefix}base_link_joint" type="fixed">
-      <xacro:insert_block name="origin" />
-      <parent link="${parent}" />
-      <child link="${tf_prefix}base_link" />
+      <xacro:insert_block name="origin"></xacro:insert_block>
+      <parent link="${parent}"></parent>
+      <child link="${tf_prefix}base_link"></child>
     </joint>
     <link name="${tf_prefix}base_link">
-      <collision name="${tf_prefix}base_link_collision">
-        <origin rpy="0.00000 0.00000 0.00000" xyz="0.00000 0.00000 0.00000" />
+      <inertial>
+        <origin rpy="0 0 0" xyz="0.00078073 -0.005657 0.036649"></origin>
+        <mass value="0.61398"></mass>
+        <inertia ixx="0.0015423" ixy="2.1048E-05" ixz="-2.1541E-06" iyy="0.0014689" iyz="7.0187E-07" izz="0.0015067"></inertia>
+      </inertial>
+      <visual>
+        <origin rpy="0 0 0" xyz="0 0 0"></origin>
         <geometry>
-          <mesh filename="file://$(find rbs_arm)/meshes/collision/start_link.stl"
-            scale="1.00000 1.00000 1.00000" />
+          <mesh filename="file://$(find rbs_arm)/meshes/visual/base_link.stl"></mesh>
+        </geometry>
+        <material name="">
+          <color rgba="0.75294 0.75294 0.75294 1"></color>
+        </material>
+      </visual>
+      <collision>
+        <origin rpy="0 0 0" xyz="0 0 0"></origin>
+        <geometry>
+          <mesh filename="file://$(find rbs_arm)/meshes/collision/base_link.stl"></mesh>
         </geometry>
       </collision>
-      <inertial>
-        <inertia ixx="0.00503302470272442" ixy="0.000343817346410954" ixz="-4.74990755448368E-06"
-          iyy="0.00337962410057753" iyz="-2.3099255620051E-05" izz="0.00405858207282473" />
-        <origin rpy="0.00000 0.00000 0.00000"
-          xyz="-0.000297002857922682 0.0964721185617698 -0.000361033370053684" />
-        <mass value="1.88031044620482" />
-      </inertial>
-      <visual name="${tf_prefix}base_link_visual">
-        <origin rpy="0.00000 0.00000 0.00000" xyz="0.00000 0.00000 0.00000" />
-        <geometry>
-          <mesh filename="file://$(find rbs_arm)/meshes/visual/start_link.dae"
-            scale="1.00000 1.00000 1.00000" />
-        </geometry>
-      </visual>
     </link>
     <!-- <xacro:joint_hardware joint_name="${tf_prefix}base_link" hardware="${hardware}" p="100"/> -->
-    <xacro:rbs_materials link_name="${tf_prefix}base_link" link_type="base_link" />
+    <!-- <xacro:rbs_materials link_name="${tf_prefix}base_link" link_type="base_link"></xacro:rbs_materials> -->
   </xacro:macro>
 </robot>

File: urdf/inc/rbs_ee_link.xacro (robot description, xacro)
@@ -1,16 +1,16 @@
 <?xml version="1.0" encoding="UTF-8"?>
 <robot xmlns:xacro="http://www.ros.org/wiki/xacro">
-  <xacro:macro name="ee_link" params="tf_prefix parent hardware p d">
+  <xacro:macro name="ee_link" params="tf_prefix parent hardware p d initial_joint_position:=^|0.0">
     <xacro:include filename="$(find rbs_arm)/urdf/inc/joint_hardware.xacro" />
     <xacro:include filename="$(find rbs_arm)/urdf/inc/materials.xacro" />
     <joint name="${tf_prefix}ee_link_joint" type="revolute">
-      <limit lower="-1.5708" upper="3.14159" effort="78" velocity="0.52" />
-      <origin rpy="0.00000 0.00000 0.00000" xyz="0.10000 0.00000 0.09473" />
+      <limit lower="-2.43" upper="2.43" effort="78" velocity="0.52" />
+      <origin rpy="0 0 0.0" xyz="0.0 0.0 0.0754"></origin>
       <parent link="${tf_prefix}${parent}" />
       <child link="${tf_prefix}ee_link" />
-      <axis xyz="0 1 0" />
+      <axis xyz="0 0 1" />
     </joint>
     <joint name="${tf_prefix}tool0_joint" type="fixed">
-      <origin rpy="0.00000 0.00000 0.00000" xyz="0.00000 0.00000 0.11000" />
+      <origin rpy="0.00000 0.00000 0.00000" xyz="0.00000 0.00000 0.14100" />
       <parent link="${tf_prefix}ee_link" />
       <child link="${tf_prefix}tool0" />
@@ -18,28 +18,29 @@
     <link name="${tf_prefix}tool0" />
     <link name="${tf_prefix}ee_link">
-      <collision name="${tf_prefix}ee_link_collision">
-        <origin rpy="-0.00000 0.00000 -0.00000" xyz="0.00000 -0.00000 0.00000" />
+      <inertial>
+        <origin rpy="0 0 0" xyz="1.594E-06 0.085889 0.0021969"></origin>
+        <mass value="0.20976"></mass>
+        <inertia ixx="0.00016257" ixy="4.2628E-07" ixz="-3.8857E-07" iyy="0.00022468"
+          iyz="2.1709E-05" izz="0.00023702"></inertia>
+      </inertial>
+      <visual>
+        <origin rpy="0 0 0" xyz="0 0 0"></origin>
         <geometry>
-          <mesh filename="file://$(find rbs_arm)/meshes/collision/ee_link.stl"
-            scale="1.00000 1.00000 1.00000" />
+          <mesh filename="file://$(find rbs_arm)/meshes/visual/axis7_tail.stl"></mesh>
+        </geometry>
+        <material name="">
+          <color rgba="0.75294 0.75294 0.75294 1"></color>
+        </material>
+      </visual>
+      <collision>
+        <origin rpy="0 0 0" xyz="0 0 0"></origin>
+        <geometry>
+          <mesh filename="file://$(find rbs_arm)/meshes/collision/axis7_tail.stl"></mesh>
         </geometry>
       </collision>
-      <inertial>
-        <inertia ixx="0.00147695259043549" ixy="-2.66894744420299E-05" ixz="-4.40871314563273E-05"
-          iyy="0.00135500487881796" iyz="-3.19001462979333E-05" izz="0.00087582892706912" />
-        <origin rpy="0.00000 0.00000 0.00000"
-          xyz="-9.7531539777207E-06 -0.000888494418875867 0.0342332199538358" />
-        <mass value="1.88031044620482" />
-      </inertial>
-      <visual name="${tf_prefix}ee_link_visual">
-        <origin rpy="0.00000 0.00000 0.00000" xyz="0.00000 -0.00000 0.00000" />
-        <geometry>
-          <mesh filename="file://$(find rbs_arm)/meshes/visual/ee_link.dae"
-            scale="1.00000 1.00000 1.00000" />
-        </geometry>
-      </visual>
     </link>
-    <xacro:joint_hardware joint_name="${tf_prefix}ee_link_joint" hardware="${hardware}" p="${p}" d="${d}" />
-    <xacro:rbs_materials link_name="${tf_prefix}ee_link" link_type="ee_link" />
+    <xacro:joint_hardware joint_name="${tf_prefix}ee_link_joint" hardware="${hardware}" p="${p}"
+      d="${d}" initial_joint_position="${initial_joint_position}" />
+    <!-- <xacro:rbs_materials link_name="${tf_prefix}ee_link" link_type="ee_link" /> -->
   </xacro:macro>
 </robot>

File: urdf/inc/rbs_fork_link.xacro (robot description, xacro)
@@ -1,5 +1,6 @@
 <?xml version="1.0" encoding="UTF-8"?>
 <robot xmlns:xacro="http://www.ros.org/wiki/xacro">
-  <xacro:macro name="fork_link" params="tf_prefix parent name hardware p d">
+  <xacro:macro name="fork_link"
+    params="tf_prefix parent name hardware p d initial_joint_position:=^|0.0">
     <xacro:include filename="$(find rbs_arm)/urdf/inc/joint_hardware.xacro" />
     <xacro:include filename="$(find rbs_arm)/urdf/inc/materials.xacro" />
@@ -7,8 +8,8 @@
       <limit lower="-6.14159" upper="6.14159" effort="78" velocity="0.52" />
       <xacro:if value="${parent=='base_link'}">
-        <origin rpy="0.00000 0.00000 0.00000" xyz="0.00000 0.00000 0.17833" />
+        <origin rpy="0.0 0 -3.1416" xyz="0 0 0.11165"></origin>
       </xacro:if>
       <xacro:unless value="${parent=='base_link'}">
-        <origin rpy="0.00000 0.00000 0.00000" xyz="0.00000 0.00000 0.13300" />
+        <origin rpy="0 0 0" xyz="0.0 0.0 0.11995"></origin>
       </xacro:unless>
       <parent link="${tf_prefix}${parent}" />
@@ -17,28 +18,29 @@
     </joint>
     <link name="${tf_prefix}${name}">
-      <collision name="${tf_prefix}${name}_collision">
-        <origin rpy="0.00000 0.00000 0.00000" xyz="0.00000 -0.00000 0.00000" />
+      <inertial>
+        <origin rpy="0 0 0" xyz="-0.0050017 0.088736 0.0023758"></origin>
+        <mass value="0.49312"></mass>
+        <inertia ixx="0.0016921" ixy="-1.8404E-05" ixz="9.951E-07" iyy="0.00087841"
+          iyz="-2.5874E-06" izz="0.0019955"></inertia>
+      </inertial>
+      <visual>
+        <origin rpy="0 0 0" xyz="0 0 0"></origin>
         <geometry>
-          <mesh filename="file://$(find rbs_arm)/meshes/collision/fork_link.stl"
-            scale="1.00000 1.00000 1.00000" />
+          <mesh filename="file://$(find rbs_arm)/meshes/visual/axis1_fork.stl"></mesh>
+        </geometry>
+        <material name="">
+          <color rgba="0.75294 0.75294 0.75294 1"></color>
+        </material>
+      </visual>
+      <collision>
+        <origin rpy="0 0 0" xyz="0 0 0"></origin>
+        <geometry>
+          <mesh filename="file://$(find rbs_arm)/meshes/collision/axis1_fork.stl"></mesh>
         </geometry>
       </collision>
-      <inertial>
-        <inertia ixx="0.00367804533572758" ixy="1.04277925521833E-05" ixz="-0.00149971410403071"
-          iyy="0.00415208849477534" iyz="-0.00122" izz="0.00329" />
-        <origin rpy="0.00000 0.00000 0.00000"
-          xyz="0.0472051139085306 0.00208890925682996 0.0557265410642575" />
-        <mass value="1.12472202892859" />
-      </inertial>
-      <visual name="${tf_prefix}${name}_visual">
-        <origin rpy="0.00000 -0.00000 -0.00000" xyz="0.00000 -0.00000 0.00000" />
-        <geometry>
-          <mesh filename="file://$(find rbs_arm)/meshes/visual/fork_link.dae"
-            scale="1.00000 1.00000 1.00000" />
-        </geometry>
-      </visual>
     </link>
-    <xacro:joint_hardware joint_name="${tf_prefix}${name}_joint" hardware="${hardware}" p="${p}" d="${d}" />
-    <xacro:rbs_materials link_name="${tf_prefix}${name}" link_type="fork" />
+    <xacro:joint_hardware joint_name="${tf_prefix}${name}_joint" hardware="${hardware}" p="${p}"
+      d="${d}" initial_joint_position="${initial_joint_position}" />
+    <!-- <xacro:rbs_materials link_name="${tf_prefix}${name}" link_type="fork" /> -->
   </xacro:macro>
 </robot>

File: urdf/inc/rbs_main_link.xacro (robot description, xacro)
@@ -1,40 +1,42 @@
 <?xml version="1.0" encoding="UTF-8"?>
 <robot xmlns:xacro="http://www.ros.org/wiki/xacro">
-  <xacro:macro name="main_link" params="tf_prefix parent name hardware p d">
+  <xacro:macro name="main_link"
+    params="tf_prefix parent name hardware p d initial_joint_position:=^|0.0">
     <xacro:include filename="$(find rbs_arm)/urdf/inc/joint_hardware.xacro" />
     <xacro:include filename="$(find rbs_arm)/urdf/inc/materials.xacro" />
     <joint name="${tf_prefix}${name}_joint" type="revolute">
-      <limit lower="-1.5708" upper="3.14159" effort="78" velocity="0.52" />
-      <origin rpy="-0.00000 0.00000 0.00000" xyz="0.10000 0.00000 0.09400" />
+      <limit lower="-2.43" upper="2.43" effort="78" velocity="0.52" />
+      <!-- <origin rpy="0.0 0 -3.1416" xyz="0 0 0.11165"></origin> -->
+      <origin rpy="0.0 0 0" xyz="0 0.0 0.15465"></origin>
       <parent link="${tf_prefix}${parent}" />
       <child link="${tf_prefix}${name}" />
-      <axis xyz="0 1 0" />
+      <axis xyz="1 0 0" />
     </joint>
     <link name="${tf_prefix}${name}">
-      <collision name="${tf_prefix}${name}_collision">
-        <origin rpy="0.00000 0.00000 0.00000" xyz="0.00000 0.00000 0.00000" />
+      <inertial>
+        <origin rpy="0 0 0" xyz="0.00027998 -0.045366 0.0068959"></origin>
+        <mass value="0.42726"></mass>
+        <inertia ixx="0.0013794" ixy="-4.0542E-05" ixz="-8.9181E-06" iyy="0.00047255"
+          iyz="-3.4771E-05" izz="0.001587"></inertia>
+      </inertial>
+      <visual>
+        <origin rpy="0 0 0" xyz="0 0 0"></origin>
         <geometry>
-          <mesh filename="file://$(find rbs_arm)/meshes/collision/main_link.stl"
-            scale="1.00000 1.00000 1.00000" />
+          <mesh filename="file://$(find rbs_arm)/meshes/visual/axis2_main.stl"></mesh>
+        </geometry>
+        <material name="">
+          <color rgba="0.75294 0.75294 0.75294 1"></color>
+        </material>
+      </visual>
+      <collision>
+        <origin rpy="0 0 0" xyz="0 0 0"></origin>
+        <geometry>
+          <mesh filename="file://$(find rbs_arm)/meshes/collision/axis2_main.stl"></mesh>
         </geometry>
       </collision>
-      <inertial>
-        <inertia ixx="0.00315699373090845" ixy="2.84713820858537E-05" ixz="-7.01601261191721E-05"
-          iyy="0.00343729241263707" iyz="-0.000101485203138902" izz="0.00125534890134052" />
-        <origin rpy="0.00000 0.00000 0.00000"
-          xyz="0.00186712264682627 -0.000412152188777604 0.0516389446895805" />
-        <mass value="1.58688811563124" />
-      </inertial>
-      <visual name="${tf_prefix}${name}_visual">
-        <origin rpy="0.00000 -0.00000 -0.00000" xyz="0.00000 0.00000 0.00000" />
-        <geometry>
-          <mesh filename="file://$(find rbs_arm)/meshes/visual/main_link.dae"
-            scale="1.00000 1.00000 1.00000" />
-        </geometry>
-      </visual>
     </link>
-    <xacro:joint_hardware joint_name="${tf_prefix}${name}_joint" hardware="${hardware}"
-      p="${p}" d="${d}" />
-    <xacro:rbs_materials link_name="${tf_prefix}${name}" link_type="main_link" />
+    <xacro:joint_hardware joint_name="${tf_prefix}${name}_joint" hardware="${hardware}" p="${p}"
+      d="${d}" initial_joint_position="${initial_joint_position}" />
+    <!-- <xacro:rbs_materials link_name="${tf_prefix}${name}" link_type="main_link" /> -->
   </xacro:macro>
 </robot>
