Commit message: Migrate to new robot structure, refactor URDF, and update GazeboSim launch
- Transitioned to a new robot structure with updated URDF and Xacro definitions.
- Updated `rbs_ee_link.xacro`, `rbs_fork_link.xacro`, and `rbs_main_link.xacro`:
  - Adjusted joint limits, positions, and axes.
  - Standardized joint parameters and transformations.
  - Updated inertia, mass, and mesh references.
  - Added `initial_joint_position` for better initialization.
- Refactored `rbs_arm_modular_macro.xacro`:
  - Simplified link definitions and removed legacy gripper integration.
  - Improved Gazebo compatibility.
- Updated `sensors.xacro` to use `gz_ros2_control/GzFts` instead of `IgnitionFts`.
- Removed outdated URDF files (`rbs_arm.urdf`, `rbs_arm.xacro`, etc.).
- Refactored `display_gazebosim.launch.py`:
  - Introduced `OpaqueFunction` and `load_xacro_args` for improved launch setup.
  - Enhanced robot description processing using `xacro.process_file`.
  - Added a clock bridge node for time synchronization.
- Updated URDF/Xacro files:
  - Introduced `initial_joint_position` in `joint_hardware.xacro` and `joint_interface.xacro`.
  - Refactored `rbs_base_link.xacro` for improved formatting and efficiency.
- Modified collision and visual mesh files:
  - Added new STL files for individual axes and base link.
  - Removed outdated STL files (`ee_link.stl`, `fork_link.stl`, etc.).

File: urdf/rbs_arm_modular_macro.xacro (robot description, xacro)
@@ -1,42 +1,33 @@
 <?xml version="1.0" encoding="UTF-8"?>
 <robot xmlns:xacro="http://www.ros.org/wiki/xacro">
-  <xacro:macro name="rbs_arm"
-    params="namespace parent *origin tf_prefix hardware gripper_name controllers">
-    <xacro:include filename="$(find rbs_arm)/urdf/inc/rbs_base_link.xacro" />
-    <xacro:include filename="$(find rbs_arm)/urdf/inc/rbs_ee_link.xacro" />
-    <xacro:include filename="$(find rbs_arm)/urdf/inc/rbs_fork_link.xacro" />
-    <xacro:include filename="$(find rbs_arm)/urdf/inc/rbs_main_link.xacro" />
-    <xacro:include filename="$(find rbs_arm)/urdf/sensors.xacro" />
+  <xacro:macro name="rbs_arm" params="namespace parent *origin tf_prefix hardware gripper_name controllers">
+    <xacro:include filename="$(find rbs_arm)/urdf/inc/rbs_base_link.xacro"></xacro:include>
+    <xacro:include filename="$(find rbs_arm)/urdf/inc/rbs_ee_link.xacro"></xacro:include>
+    <xacro:include filename="$(find rbs_arm)/urdf/inc/rbs_fork_link.xacro"></xacro:include>
+    <xacro:include filename="$(find rbs_arm)/urdf/inc/rbs_main_link.xacro"></xacro:include>
+    <xacro:include filename="$(find rbs_arm)/urdf/sensors.xacro"></xacro:include>
     <!-- BEGIN robot description  -->
-    <xacro:base_link parent="${parent}" tf_prefix="${tf_prefix}" hardware="${hardware}">
-      <xacro:insert_block name="origin" />
+    <xacro:base_link hardware="${hardware}" parent="${parent}" tf_prefix="${tf_prefix}">
+      <xacro:insert_block name="origin"></xacro:insert_block>
     </xacro:base_link>
-    <xacro:fork_link parent="base_link" name="fork0_link" tf_prefix="${tf_prefix}"
-      hardware="${hardware}" p="10000" d="0.2" />
-    <xacro:main_link parent="fork0_link" name="main0_link" tf_prefix="${tf_prefix}"
-      hardware="${hardware}"
-      p="10000" d="0.2" />
-    <xacro:fork_link parent="main0_link" name="fork1_link" tf_prefix="${tf_prefix}"
-      hardware="${hardware}" p="10000" d="0.2" />
-    <xacro:main_link parent="fork1_link" name="main1_link" tf_prefix="${tf_prefix}"
-      hardware="${hardware}" p="1000" d="0.2" />
-    <xacro:fork_link parent="main1_link" name="fork2_link" tf_prefix="${tf_prefix}"
-      hardware="${hardware}" p="100" d="0.2" />
+    <xacro:fork_link d="0.2" hardware="${hardware}" name="fork0_link" p="10000" parent="base_link" tf_prefix="${tf_prefix}"></xacro:fork_link>
+    <xacro:main_link d="0.2" hardware="${hardware}" name="main0_link" p="10000" parent="fork0_link" tf_prefix="${tf_prefix}"></xacro:main_link>
+    <xacro:fork_link d="0.2" hardware="${hardware}" name="fork1_link" p="10000" parent="main0_link" tf_prefix="${tf_prefix}"></xacro:fork_link>
+    <xacro:main_link d="0.2" hardware="${hardware}" name="main1_link" p="1000" parent="fork1_link" tf_prefix="${tf_prefix}"></xacro:main_link>
+    <xacro:fork_link d="0.2" hardware="${hardware}" name="fork2_link" p="100" parent="main1_link" tf_prefix="${tf_prefix}"></xacro:fork_link>
+    <xacro:main_link d="0.2" hardware="${hardware}" name="main2_link" p="1000" parent="fork2_link" tf_prefix="${tf_prefix}"></xacro:main_link>
     <!-- ee link also contain tool0-->
-    <xacro:ee_link parent="fork2_link" tf_prefix="${tf_prefix}" hardware="${hardware}"
-      p="20" d="0.2" />
+    <xacro:ee_link d="0.2" hardware="${hardware}" p="20" parent="main2_link" tf_prefix="${tf_prefix}"></xacro:ee_link>
     <!-- END robot description -->
     <!-- Insert gripper in robot description if exist -->
-    <xacro:if value="${gripper_name=='rbs_gripper'}">
-      <xacro:include filename="$(find rbs_gripper)/urdf/rbs_gripper_macro.xacro" />
-      <xacro:rbs_gripper tf_prefix="${tf_prefix}" gripper_name="rbs_gripper"
-        parent="${tf_prefix}tool0"
-        hardware="${hardware}">
-        <origin xyz="0.0 0.0 0.0" rpy="0.0 0.0 0.0" />
-      </xacro:rbs_gripper>
-    </xacro:if>
+    <!-- <xacro:if value="${gripper_name=='rbs_gripper'}"> -->
+    <!--   <xacro:include filename="$(find rbs_gripper)/urdf/rbs_gripper_macro.xacro"></xacro:include> -->
+    <!--   <xacro:rbs_gripper gripper_name="rbs_gripper" hardware="${hardware}" parent="${tf_prefix}tool0" tf_prefix="${tf_prefix}"> -->
+    <!--     <origin rpy="0.0 0.0 0.0" xyz="0.0 0.0 0.0"></origin> -->
+    <!--   </xacro:rbs_gripper> -->
+    <!-- </xacro:if> -->
     <!-- If hardware == gazebo so insert additional parameters for it -->
     <xacro:if value="${hardware=='gazebo'}">
-      <xacro:fts name="fts_sensor" tf_prefix="${tf_prefix}" link="${tf_prefix}tool0" />
+      <!-- <xacro:fts link="tool0" name="fts_sensor" tf_prefix="${tf_prefix}"></xacro:fts> -->
       <gazebo>
         <plugin filename="gz_ros2_control-system" name="gz_ros2_control::GazeboSimROS2ControlPlugin">

File: urdf/sensors.xacro (robot description, xacro)
@@ -54,5 +54,5 @@
     <ros2_control name="${tf_prefix}${name}" type="sensor">
       <hardware>
-          <plugin>ign_ros2_control/IgnitionFts</plugin>
+          <plugin>gz_ros2_control/GzFts</plugin>
       </hardware>
       <sensor name="${tf_prefix}${name}">

Commit message: delete p and d coeffs in ros2_control interface

File: urdf/inc/joint_hardware.xacro (robot description, xacro)
@@ -3,5 +3,5 @@
   <xacro:include filename="$(find rbs_arm)/urdf/inc/joint_interface.xacro" />
   <xacro:macro name="joint_hardware"
-    params="joint_name hardware p:=^ d:=^ initial_joint_position:=^|0.0">
+    params="joint_name hardware initial_joint_position:=^|0.0">
     <ros2_control name="${joint_name}_hardware_interface" type="actuator">
       <hardware>
@@ -13,5 +13,5 @@
         </xacro:if>
       </hardware>
-      <xacro:joint_interface name="${joint_name}" p="${p}" d="${d}"
+      <xacro:joint_interface name="${joint_name}"
         initial_joint_position="${initial_joint_position}" />
     </ros2_control>

File: urdf/inc/joint_interface.xacro (robot description, xacro)
@@ -2,12 +2,8 @@
 <robot xmlns:xacro="http://www.ros.org/wiki/xacro">
   <!-- Individual joint. -->
-  <xacro:macro name="joint_interface" params="name p:=^ d:=^ initial_joint_position:=^|0.0">
+  <xacro:macro name="joint_interface" params="name initial_joint_position:=^|0.0">
     <joint name="${name}">
       <command_interface name="position" />
       <command_interface name="velocity" />
-      <!-- WARN When this active a robot falls down -->
-      <!-- <command_interface name="effort"/> -->
-      <param name="p">${p}</param>
-      <param name="d">${d}</param>
       <!-- <command_interface name="effort"/> -->
       <state_interface name="position">
