Commit message: update urdf

File: urdf/rbs_arm.urdf (robot description, URDF)
Before this commit: robot rbs_arm, 9 links, 8 joints
Links:
- added link gripper_grasp_point
- added link rbs_gripper_gripper_base_link, mass 1.13983632906086; collision mesh filename=file:///home/bill-finger/rbs_ws/install/rbs_gripper/share/r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; visual mesh filename=file:///home/bill-finger/rbs_ws/install/rbs_gripper/share/r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
- added link rbs_gripper_l_finger_link, mass 0.0601996441483964; collision mesh filename=file:///home/bill-finger/rbs_ws/install/rbs_gripper/share/r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; visual mesh filename=file:///home/bill-finger/rbs_ws/install/rbs_gripper/share/r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
- added link rbs_gripper_r_finger_link, mass 0.0602; collision mesh filename=file:///home/bill-finger/rbs_ws/install/rbs_gripper/share/r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; visual mesh filename=file:///home/bill-finger/rbs_ws/install/rbs_gripper/share/r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
- added link rbs_gripper_rot_base_link, mass 0.161003401535982; collision mesh filename=file:///home/bill-finger/rbs_ws/install/rbs_gripper/share/r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; visual mesh filename=file:///home/bill-finger/rbs_ws/install/rbs_gripper/share/r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
Joints:
- added joint rbs_gripper_gripper_base_joint: type fixed, parent tool0, child rbs_gripper_gripper_base_link, origin xyz=0 0 0 rpy=0 0 0
- added joint rbs_gripper_gripper_tool0_joint: type fixed, parent rbs_gripper_rot_base_link, child gripper_grasp_point, origin xyz=0 0 0.09139 rpy=0 0 0
- added joint rbs_gripper_l_finger_joint: type prismatic, parent rbs_gripper_rot_base_link, child rbs_gripper_l_finger_link, origin xyz=0 0 0.1071 rpy=0 0 1.5708, axis -1 0 0, limit lower=0 upper=0.064 effort=10 velocity=0.53, mimic joint=rbs_gripper_r_finger_joint multiplier=1
- added joint rbs_gripper_r_finger_joint: type prismatic, parent rbs_gripper_rot_base_link, child rbs_gripper_r_finger_link, origin xyz=0 0 0.1071 rpy=0 0 -1.5708, axis -1 0 0, limit lower=0 upper=0.064 effort=10 velocity=0.53
- added joint rbs_gripper_rot_base_joint: type revolute, parent rbs_gripper_gripper_base_link, child rbs_gripper_rot_base_link, origin xyz=0 0 0.10861 rpy=0 0 0, axis 0 0 1, limit lower=-3.14159 upper=3.14159 effort=78 velocity=0.52
- joint base_link_joint: origin xyz=0 0 0 rpy=0 0 0 -> xyz=0.0 0.0 0.0 rpy=0.0 0.0 0.0
- joint fork0_link_joint: limit lower=-3.14159 upper=3.14159 effort=78 velocity=0.52 -> lower=-6.14159 upper=6.14159 effort=78 velocity=0.52
- joint fork1_link_joint: limit lower=-3.14159 upper=3.14159 effort=78 velocity=0.52 -> lower=-6.14159 upper=6.14159 effort=78 velocity=0.52
- joint fork2_link_joint: limit lower=-3.14159 upper=3.14159 effort=78 velocity=0.52 -> lower=-6.14159 upper=6.14159 effort=78 velocity=0.52
