Commit message: rename fts sensor

File: urdf/rbs_arm_modular_macro.xacro (robot description, xacro)
@@ -35,5 +35,5 @@
     <!-- If hardware == gazebo so insert additional parameters for it -->
     <xacro:if value="${hardware=='gazebo'}">
-      <xacro:rbs_fts name="fts_sensor" tf_prefix="${tf_prefix}" link="${tf_prefix}tool0"/>
+      <xacro:fts name="fts_sensor" tf_prefix="${tf_prefix}" link="${tf_prefix}tool0"/>
       <gazebo>
         <plugin filename="libign_ros2_control-system.so"

File: urdf/sensors.xacro (robot description, xacro)
@@ -51,5 +51,5 @@
         </joint>
     </xacro:macro>
-    <xacro:macro name="rbs_fts" params="name tf_prefix link">
+    <xacro:macro name="fts" params="name tf_prefix link">
     <ros2_control name="${tf_prefix}${name}" type="sensor">
       <hardware>
